File: hardware/kicad_project/untitled.kicad_sch (KiCad schematic)
At the start: 84 parts, among them SW1 ESC, SW10 F6, SW11 F7, SW12 F8, SW13 F9, SW14 F10, SW15 F11, SW16 F12, SW17 3 #, SW18 4 $ ;, SW19 5 %, SW2 F1, SW20 6 ^ :, SW21 7 & ?, SW22 8 *, SW23 9 (, SW24 0 ), SW25 UP, SW26 DOWN, SW27 LEFT, SW28 RIGHT, SW29 INSERT, SW3 F2, SW30 HOME, SW31 PG DN, SW32 DELETE, SW33 - _, SW34 + =, SW35 | \ /, SW36 BSP, SW37 TAB, SW38 Q, SW39 W, SW4 F3, SW40 E, SW41 END, SW42 PG UP, SW43 PRNT SCRN, SW44 R, SW45 T, SW46 Y, SW47 U, SW48 I, SW49 O, SW5 F4, SW50 P, SW51 { [, SW52 } ], SW53 ENTER, SW54 CAPS, SW55 A, SW56 S, SW57 D, SW58 F, SW59 G, SW6 ` ~, SW60 H, SW61 J, SW62 K, SW63 L, SW64 : ;, SW65 " ', SW66 LSHIFT, SW67 Z, SW68 X, SW69 C, SW7 1 !, SW70 V, SW71 B, SW72 N, SW73 M, SW74 < ,, SW75 > ., SW76 / ?, SW77 RSHIFT, SW78 LCTRL, SW79 LALT, SW8 2 @ ", SW80 SPACE, SW81 RALT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

Commit message: Add files via upload
Parts:
- removed SW68: X, Button_Switch_THT:SW_PUSH_6mm_H4.3mm, symbol Switch:SW_Push
- removed SW69: C, Button_Switch_THT:SW_PUSH_6mm_H4.3mm, symbol Switch:SW_Push
- removed SW70: V, Button_Switch_THT:SW_PUSH_6mm_H4.3mm, symbol Switch:SW_Push
- removed SW71: B, Button_Switch_THT:SW_PUSH_6mm_H4.3mm, symbol Switch:SW_Push
- removed SW72: N, Button_Switch_THT:SW_PUSH_6mm_H4.3mm, symbol Switch:SW_Push
- removed SW73: M, Button_Switch_THT:SW_PUSH_6mm_H4.3mm, symbol Switch:SW_Push
- removed SW74: < ,, Button_Switch_THT:SW_PUSH_6mm_H4.3mm, symbol Switch:SW_Push
- removed SW75: > ., Button_Switch_THT:SW_PUSH_6mm_H4.3mm, symbol Switch:SW_Push
- removed SW76: / ?, Button_Switch_THT:SW_PUSH_6mm_H4.3mm, symbol Switch:SW_Push
- removed SW77: RSHIFT, Button_Switch_THT:SW_PUSH_6mm_H4.3mm, symbol Switch:SW_Push
- removed SW78: LCTRL, Button_Switch_THT:SW_PUSH_6mm_H4.3mm, symbol Switch:SW_Push
- removed SW79: LALT, Button_Switch_THT:SW_PUSH_6mm_H4.3mm, symbol Switch:SW_Push
- removed SW80, SW84: SPACE, Button_Switch_THT:SW_PUSH_6mm_H4.3mm, symbol Switch:SW_Push
- removed SW81: RALT, Button_Switch_THT:SW_PUSH_6mm_H4.3mm, symbol Switch:SW_Push
- removed SW82: RCTRL, Button_Switch_THT:SW_PUSH_6mm_H4.3mm, symbol Switch:SW_Push
- removed SW83: PAUSE, Button_Switch_THT:SW_PUSH_6mm_H4.3mm, symbol Switch:SW_Push

Commit message: Iteration 2
Parts:
- SW1: value ESC -> ОТМ
