File: hardware/kicad_project/keyb.kicad_pcb (KiCad board)
At the start: 2 copper layers, 174 x 80 mm, 120 parts, among them J1 PS/2, J2 РПрог, J3 2Мк, J4 1Мк, SW1 ОТМ, SW10 Ф6, SW11 Ф7, SW12 Ф8, SW13 Ф9, SW14 Ф10, SW15 Ф11, SW16 Ф12, SW17 3 # Нм, SW18 4 $ ;, SW19 5 %, SW2 Ф1, SW20 6 ^ :, SW21 7 & ?, SW22 8 *, SW23 9 (, SW24 0 ), SW25 ВВЕРХ, SW26 ВНИЗ, SW27 ВЛЕВО, SW28 ВПРАВО, SW29 ВСТ, SW3 Ф2, SW30 НАЗАД, SW31 СТР ВНИЗ, SW32 УД.ВП., SW33 - _, SW34 + =, SW35 \ |, SW36 УДАЛ, SW37 ТАБ, SW38 Q Й, SW39 W Ц, SW4 Ф3, SW40 E У, SW41 В КОНЕЦ, SW42 СТР ВВЕРХ, SW43 ПЕЧАТЬ, SW44 R К, SW45 T Е, SW46 Y Н, SW47 U Г, SW48 I Ш, SW49 O Щ, SW5 Ф4, SW50 P З, SW51 [ Х, SW52 ] Ъ, SW53 ВВОД, SW54 ВЕРХ.Рег, SW55 A Ф, SW56 S Ы, SW57 D В, SW58 F А, SW59 G П, SW6 ~ ` Ё, SW60 H Р, SW61 J О, SW62 K Л, SW63 L Д, SW64 : ; Ж, SW65 " ' Э, SW66 СДВГ, SW67 Z Я, SW68 X Ч, SW69 C, SW7 1 !, SW70 V М, SW71 B И, SW72 N Т, SW73 M Ь, SW74 < , Б, SW75 > . Ю, SW76 / ? ., SW77 СДВГ, SW78 КТРЛ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

Commit message: Iteration 2
Parts:
- removed J3: 2Мк, Connector_PinSocket_2.54mm:SolderJumper-2_P1.3mm_Open_RoundedPad1.0x1.5mm
- removed J4: 1Мк, Connector_PinSocket_2.54mm:SolderJumper-2_P1.3mm_Open_RoundedPad1.0x1.5mm
- removed REF**: USSRQ, Symbol:USSRQ
- removed RN2: 10K, Resistor_THT:R_Array_SIP9
- removed Ue1: К555ИР9 - 2, Package_DIP:DIP-16_W7.62mm_Socket
- D1: value Св1 -> Св.1
- D2: value Св2 -> Св.2
- J2: value РПрог -> ICSP
- SW17: value 3 # Нм -> 3 #
- SW29: value ВСТ -> ВСТВ
- SW32: value УД.ВП. -> УД. ВП.
- SW51: value [ Х -> [ X {
- SW52: value ] Ъ -> ] Ъ }
- SW54: value ВЕРХ.Рег -> ВЕРХРег
- SW6: value ~ ` Ё -> ` ~ Ё
- SW65: value " ' Э -> ' " Э
- SW66: value СДВГ -> LSHIFT
- SW77: value СДВГ -> RSHIFT
- U1: value ATtiny2313A -> ATtiny2313-20P
- U2: value КР1564ИР52- 1 -> KP1564ИP52 - 1
- U3: value КР1564ИР52 - 2 -> KP1564ИP52- 2
- U4: value К555ИР9 - 1 -> KP1564ИP9
- moved RN1 13.6 mm to (160.0, 81.8)
- moved U4 7.65 mm to (137.2, 84.1)
- moved U2 4.39 mm to (89.9, 84.1)
- moved U3 4.39 mm to (111.9, 84.1)
- moved J2 2.15 mm to (83.4, 77.3)
Connections:
- U4 pad 10: Net-(J3-Pad2) -> GND
Routing:
- net PDATA: track 180.3 -> 265.1 mm, vias 2 -> 3
- net SO: track 93.6 -> 174.6 mm, vias 1 -> 2
- net Net-(J3-Pad2): track 73.6 -> 0.00 mm, vias 1 -> 0
- net PCLK: track 218.8 -> 152.9 mm
- net Net-(D2-A): track 205.0 -> 252.3 mm
- net shft: track 46.1 -> 0.00 mm
- net KL4_595: track 319.6 -> 358.8 mm, vias 1 -> 2
- net KL1_595: track 273.4 -> 234.6 mm
- net KL5_595: track 247.6 -> 212.6 mm, vias 1 -> 0
- net D12_165: track 32.5 -> 0.00 mm
- net D9_165: track 32.2 -> 0.00 mm
- net D11_165: track 32.1 -> 0.00 mm
- net D10_165: track 32.1 -> 0.00 mm
- net D8_165: track 31.6 -> 0.00 mm
- net KL7_595: track 276.8 -> 308.0 mm, vias 1 -> 0
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Other:
- board text added: "Mобильные Kибернетические Cистемы"
- board text added: "OПP CCCP 11.2023"
- board text removed: "Мобильные Кибернетические Системы"
- board text removed: "ОПР СССР 09.2022"

Commit message: Add files via upload
Routing:
- net D1_165: track 318.7 -> 322.3 mm
- net KL1_595: track 234.6 -> 236.6 mm
- net KL12_595: track 148.6 -> 150.0 mm
- net D7_165: track 316.1 -> 316.8 mm
